File: mainboard/mainboard.kicad_pcb (KiCad board)
At the start: 4 copper layers, 68 x 86.5 mm, 80 parts, among them J1 Servo, J2 Buzzer, J4 Button Interface, J5 Power, J6 Release Button, J7 Extra Pins, Q1 BSS138, Q2 BSS138, Q3 BSS138, Q4 BSS138, Q5 BSS138, Q6 BSS138, SW1 SW_Push, U1 RP2040, U2 W25Q128JVS, U3 RV-3028-C7, U4 ITR9608-F, U5 TCA9535RTWR, U6 11405, Y1 Crystal_ABM8

Commit message: ground vias
Routing:
- net GND: vias 56 -> 189
